Commit message: changing topic and frame names to be more explicit

File: src/vehicle_simulator/urdf/lidar2D.urdf.xacro (robot description, xacro)
@@ -1,5 +1,5 @@
 <?xml version="1.0"?>
 <robot xmlns:xacro="http://www.ros.org/wiki/xacro" name="lidar2d_robot">
-  <link name="lidar_holder2D">
+  <link name="lidar2D_frame">
     <collision>
       <origin xyz="0 0 0" rpy="0 0 0"/>
@@ -21,5 +21,5 @@
   </link>
   <!-- Gazebo plugin attached to lidar_holder2D -->
-  <gazebo reference="lidar_holder2D">
+  <gazebo reference="lidar2D_frame">
     <material>Gazebo/Red</material>
     <sensor name="laser" type="ray">
@@ -41,7 +41,7 @@
       </ray>
       <plugin name="laser_controller" filename="libgazebo_ros_laser.so">
-        <topicName>scan</topicName>
+        <topicName>lidar2D_scan</topicName>
         <output_type>sensor_msgs/LaserScan</output_type>
-        <frameName>lidar_holder2D</frameName>
+        <frameName>lidar2D_frame</frameName>
       </plugin>
     </sensor>
